File: KiCAD/TisKnob_V01-00-00/TisKnob_V01-00-00.kicad_sch (KiCad schematic)
At the start: 0 parts

Commit message: KiCAD
Parts:
- added D1, D10, D11, D12, D13, D14, D15, D16, D17, D18, D19, D2, D20, D21, D22, D23, D24, D3, D4, D5, D6, D7, D8, D9: WS2812B-2020, TouchKnob:LED_WS2812B-2020_PLCC4_2.0x2.0mm, symbol LED:WS2812B-2020
Connections:
- new net: D17.1 (DOUT), D18.3 (DIN)
- new net: D1.2 (VSS), D10.2 (VSS), D11.2 (VSS), D12.2 (VSS), D13.2 (VSS), D14.2 (VSS), D15.2 (VSS), D16.2 (VSS), D17.2 (VSS), D18.2 (VSS), D19.2 (VSS), D2.2 (VSS), D20.2 (VSS), D21.2 (VSS), D22.2 (VSS), D23.2 (VSS), D24.2 (VSS), D3.2 (VSS), D4.2 (VSS), D5.2 (VSS), D6.2 (VSS), D7.2 (VSS), D8.2 (VSS), D9.2 (VSS)
- new net: D16.1 (DOUT), D17.3 (DIN)
- new net: D1.4 (VDD), D10.4 (VDD), D11.4 (VDD), D12.4 (VDD), D13.4 (VDD), D14.4 (VDD), D15.4 (VDD), D16.4 (VDD), D17.4 (VDD), D18.4 (VDD), D19.4 (VDD), D2.4 (VDD), D20.4 (VDD), D21.4 (VDD), D22.4 (VDD), D23.4 (VDD), D24.4 (VDD), D3.4 (VDD), D4.4 (VDD), D5.4 (VDD), D6.4 (VDD), D7.4 (VDD), D8.4 (VDD), D9.4 (VDD)
- new net: D14.1 (DOUT), D15.3 (DIN)
- new net: D13.1 (DOUT), D14.3 (DIN)
- new net: D23.1 (DOUT), D24.3 (DIN)
- new net: D15.1 (DOUT), D16.3 (DIN)
- new net: D2.1 (DOUT), D3.3 (DIN)
- new net: D1.1 (DOUT), D2.3 (DIN)
- new net: D22.1 (DOUT), D23.3 (DIN)
- new net: D21.1 (DOUT), D22.3 (DIN)
- new net: D8.1 (DOUT), D9.3 (DIN)
- new net: D7.1 (DOUT), D8.3 (DIN)
- new net: D12.1 (DOUT), D13.3 (DIN)
- new net: D11.1 (DOUT), D12.3 (DIN)
- new net: D4.1 (DOUT), D5.3 (DIN)
- new net: D3.1 (DOUT), D4.3 (DIN)
- new net: D20.1 (DOUT), D21.3 (DIN)
- new net: D10.1 (DOUT), D11.3 (DIN)
- new net: D10.3 (DIN), D9.1 (DOUT)
- new net: D6.1 (DOUT), D7.3 (DIN)
- new net: D19.1 (DOUT), D20.3 (DIN)
- new net: D5.1 (DOUT), D6.3 (DIN)
- new net: D18.1 (DOUT), D19.3 (DIN)
